File: v0.8/RFM69 USB Gateway 0.8.brd (EAGLE design)
At the start: 40.7 x 17.3 mm, 25 parts, among them CN1 MINIB, IC3 MCP1703CB, U2 ATMEGA328P-MU, X1 16 MHz

Commit message: Routed all traces
Rearranged components on the board
Parts:
- R3, R5: value 27 -> 27Ω
- moved C4 12.9 mm to (32.4, 17.3), turned to 270 degrees
- moved R7 9.71 mm to (39.8, 15.9), turned to 180 degrees
- moved R2 9.31 mm to (46.3, 4.78)
- moved U$2 7.94 mm to (50.2, 4.76)
- moved C2 6.10 mm to (25.0, 17.2), turned to 270 degrees
- moved R1 5.20 mm to (33.3, 6.72)
- moved R4 5.12 mm to (28.8, 6.83)
- moved U$7 5.00 mm to (28.7, 4.69)
- moved X1 3.74 mm to (37.7, 6.72)
- moved U$4 3.61 mm to (24.0, 4.67), turned to 180 degrees
- moved R6 3.52 mm to (23.9, 6.85)
- moved IC3 2.03 mm to (28.7, 17.4)
- moved D 1.93 mm to (22.7, 17.2), turned to 270 degrees
- moved C1 1.61 mm to (30.5, 13.2)
- moved C6 1.26 mm to (20.4, 17.2), turned to 90 degrees
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Routing:
- net VCC: track 0.00 -> 67.7 mm, vias 0 -> 2
- net RESET: track 0.00 -> 31.3 mm, vias 0 -> 2
- net VBUS: track 0.00 -> 23.4 mm, vias 0 -> 2
- net N$3: track 0.00 -> 22.1 mm
- net D11_MOSI: track 0.00 -> 20.2 mm, vias 0 -> 1
- net D10_SS: track 0.00 -> 19.0 mm, vias 0 -> 2
- net D2: track 0.00 -> 18.2 mm, vias 0 -> 1
- net GND: track 0.00 -> 16.8 mm, vias 0 -> 9
- net D12_MISO: track 0.00 -> 16.3 mm
- net D13_SCK: track 0.00 -> 16.0 mm
- net N$7: track 0.00 -> 15.9 mm, vias 0 -> 2
- net FTDI3.3V: track 0.00 -> 15.8 mm, vias 0 -> 2
- net D9: track 0.00 -> 13.8 mm, vias 0 -> 2
- net D1_TX: track 0.00 -> 12.0 mm, vias 0 -> 2
- net N$6: track 0.00 -> 6.62 mm, vias 0 -> 2
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