File: v0.91/RFM69 USB Gateway 0.91.brd (EAGLE design)
At the start: 45.2 x 17 mm, 25 parts, among them IC3 MCP1703-3.3V, J1 USBPCB_NOPASTE, U2 ATMEGA328P-MU, X1 16 MHz

Commit message: Connected all traces
Parts:
- moved R2 25.7 mm to (72.0, 5.68), turned to 270 degrees
- moved U$2 23.9 mm to (74.0, 5.56), turned to 90 degrees
- moved U$1 23.3 mm to (73.9, 18.3)
- moved J$1 22.1 mm to (72.7, 9.08)
Routing:
- net D2: track 1.50 -> 46.7 mm, vias 1 -> 2
- net VCC: track 61.9 -> 100.6 mm, vias 2 -> 3
- net N$3: track 3.26 -> 36.3 mm
- net D9: track 13.8 -> 40.9 mm
- net D10_SS: track 0.93 -> 23.7 mm, vias 2 -> 3
- net D11_MOSI: track 8.09 -> 15.4 mm, vias 1 -> 2
- net D12_MISO: track 14.4 -> 18.2 mm
- net D13_SCK: track 10.0 -> 13.6 mm
- net GND: vias 20 -> 59
Other:
- board size 45.2 x 17 mm -> 68.1 x 17 mm
