File: v0.92/RFM69 USB Gateway 0.92.sch (EAGLE design)
At the start: 25 parts, among them IC3 MCP1703-3.3V, J1 USBPCB_NOPASTE, U1 RFM69HCW, U2 ATMEGA328P-MU, X1 16 MHz

Commit message: adding mpns to schematic
Parts:
- C1, C5, C6: MPN (none) -> CC0805KRX7R9BB104
- C2, C4: MPN (none) -> CC0805ZRY5V8BB105
- D: MPN (none) -> SD0805S040S0R5
- FT231XQ-R: MPN (none) -> FT231XQ-R
- IC3: MPN (none) -> MCP1703T-2502E/CB
- R1, R7: MPN (none) -> RC0805FR-0710KL
- R2: MPN (none) -> RC0805FR-071KL
- R3, R5: MPN (none) -> RC0805FR-0727RL
- R4, R6: MPN (none) -> RC0805FR-0747RL
- RX, TX, U$2: MPN (none) -> LG R971-KN-1
- U1: MPN (none) -> RFM69HW
- U2: MPN (none) -> ATMEGA328PB-AU
- X1: MPN (none) -> CSTCE16M0V53-R0
